File: src-kicad/_autosave-MPWifi_v1.kicad_pcb (KiCad board)
At the start: 2 copper layers, 16 parts, among them CON1 Micro_SD_Card, M1 ESP8266-12E, P1 CONN_01X04, P2 Flash, Q1 BSS138, Q2 BSS138, U1 MCP1703T-3302E/CB

Commit message: Netlist
Parts:
- moved P2 10.4 mm to (144.6, 69.7), turned to 180 degrees
Routing:
- net GND: track 21.2 -> 35.9 mm, vias 0 -> 2
Changed lines of the file:
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@@
   (general
     (links 48)
-    (no_connects 25)
-    (area 131.024999 52.024999 170.855 101.275001)
+    (no_connects 22)
+    (area 133.3 51.992857 174.357143 101.275001)
     (thickness 1.6)
     (drawings 0)
-    (tracks 114)
+    (tracks 124)
     (zones 0)
     (modules 16)
@@
   )
   (module Pin_Headers:Pin_Header_Angled_1x03 (layer F.Cu)
-    (at 135.5 64.7)
+    (at 144.6 69.7 180)
     (descr "Through hole pin header")
     (tags "pin header")
-    (fp_text reference P2 (at 0 -5.1) (layer F.SilkS)
-      (effects (font (size 1 1) (thickness 0.15)))
-    )
-    (fp_text value Flash (at 0 -3.1) (layer F.Fab)
+    (fp_text reference P2 (at 0 -5.1 180) (layer F.SilkS)
+      (effects (font (size 1 1) (thickness 0.15)))
+    )
+    (fp_text value Flash (at 0 -3.1 180) (layer F.Fab)
       (effects (font (size 1 1) (thickness 0.15)))
     )
@@
     (fp_line (start 1.524 1.27) (end 4.064 1.27) (layer F.SilkS) (width 0.15))
     (fp_line (start 1.524 6.35) (end 4.064 6.35) (layer F.SilkS) (width 0.15))
-    (pad 1 thru_hole rect (at 0 0) (size 2.032 1.7272) (drill 1.016) (layers *.Cu *.Mask)
+    (pad 1 thru_hole rect (at 0 0 180) (size 2.032 1.7272) (drill 1.016) (layers *.Cu *.Mask)
       (net 20 "Net-(M1-Pad12)"))
-    (pad 2 thru_hole oval (at 0 2.54) (size 2.032 1.7272) (drill 1.016) (layers *.Cu *.Mask)
+    (pad 2 thru_hole oval (at 0 2.54 180) (size 2.032 1.7272) (drill 1.016) (layers *.Cu *.Mask)
       (net 20 "Net-(M1-Pad12)"))
-    (pad 3 thru_hole oval (at 0 5.08) (size 2.032 1.7272) (drill 1.016) (layers *.Cu *.Mask)
+    (pad 3 thru_hole oval (at 0 5.08 180) (size 2.032 1.7272) (drill 1.016) (layers *.Cu *.Mask)
       (net 2 GND))
     (model Pin_Headers.3dshapes/Pin_Header_Angled_1x03.wrl
@@
   (segment (start 157.15 65.5) (end 156.58 65.5) (width 0.3) (layer B.Cu) (net 1))
   (segment (start 156.58 65.5) (end 153.93 62.85) (width 0.3) (layer B.Cu) (net 1))
+  (segment (start 151.3 80.3) (end 156.9 80.3) (width 0.76) (layer F.Cu) (net 2))
+  (segment (start 156.9 80.005) (end 157.98 78.925) (width 0.76) (layer B.Cu) (net 2))
+  (segment (start 156.9 80.3) (end 156.9 80.005) (width 0.76) (layer B.Cu) (net 2))
+  (via (at 156.9 80.3) (size 0.6) (drill 0.4) (layers F.Cu B.Cu) (net 2))
+  (segment (start 151.3 78.3) (end 150.3 77.3) (width 0.76) (layer F.Cu) (net 2))
+  (segment (start 150.3 78.475) (end 150.75 78.925) (width 0.76) (layer B.Cu) (net 2))
+  (segment (start 150.3 76.3) (end 150.3 78.475) (width 0.76) (layer B.Cu) (net 2))
+  (via (at 150.3 76.3) (size 0.6) (drill 0.4) (layers F.Cu B.Cu) (net 2))
+  (segment (start 150.3 77.3) (end 150.3 76.3) (width 0.76) (layer F.Cu) (net 2))
+  (segment (start 151.3 80.3) (end 151.3 78.3) (width 0.76) (layer F.Cu) (net 2))
   (segment (start 162.6 68.8) (end 163.45 69.65) (width 0.76) (layer F.Cu) (net 2))
   (segment (start 163.45 69.65) (end 165.2 69.65) (width 0.76) (layer F.Cu) (net 2))
@@
   (segment (start 156.47 63.28) (end 156.47 62.85) (width 0.35) (layer F.Cu) (net 2))
   (segment (start 168.6 77.5) (end 168.6 87.35) (width 0.76) (layer F.Cu) (net 3))
-  (segment (start 167.9 88.3) (end 165.3 88.3) (width 0.76) (layer F.Cu) (net 3) (status 800000))
+  (segment (start 167.9 88.3) (end 165.3 88.3) (width 0.76) (layer F.Cu) (net 3))
   (segment (start 168.6 87.6) (end 167.9 88.3) (width 0.76) (layer F.Cu) (net 3))
   (segment (start 168.6 87.35) (end 168.6 87.6) (width 0.76) (layer F.Cu) (net 3))
