File: src-kicad/MPWifi_v1.sch (KiCad schematic (older format))
At the start: 15 parts, among them CON1 Micro_SD_Card, M1 ESP8266-12E, P1 CONN_01X04, P2 Flash, Q1 BSS138, Q2 BSS138, U1 MCP1703T-3302E/CB

Commit message: Netlist
Parts:
- added R6: 10k, Resistors_SMD:R_0603, symbol R
- C1, C2: footprint (none) -> Capacitors_SMD:C_0603
- CON1: footprint 10067847-001 -> mpwifi:MicroSD-slot
- D1: footprint (none) -> Diodes_SMD:D_0603
- M1: footprint (none) -> mpwifi:ESP8266-12E
- P1: footprint (none) -> Socket_Strips:Socket_Strip_Angled_1x04
- P2: footprint (none) -> Pin_Headers:Pin_Header_Angled_1x03
- Q1, Q2: footprint SOT-23 -> TO_SOT_Packages_SMD:SOT-23
- R1: value R -> 140; footprint (none) -> Resistors_SMD:R_0603
- R2, R3, R4, R5: footprint (none) -> Resistors_SMD:R_0603
- U1: footprint SOT-223-3 -> mpwifi:SOT-223-3
Connections:
- net labels added: DETECT_SWITCH
- wire segments 71 -> 78
- no-connect marks 13 -> 12
Other:
- moved on the sheet: P1
Changed lines of the file:
@@
 LIBS:general
 LIBS:mpwifi
+LIBS:MPWifi_v1-cache
 EELAYER 25 0
 EELAYER END
@@
 F 0 "M1" H 7950 4400 60  0000 C CNN
 F 1 "ESP8266-12E" H 8250 4550 60  0000 C CNN
-F 2 "" H 8250 3950 60  0000 C CNN
+F 2 "mpwifi:ESP8266-12E" H 8250 3950 60  0001 C CNN
 F 3 "" H 8250 3950 60  0000 C CNN
 	1    8250 3950
@@
 F 0 "CON1" H 1950 5550 50  0000 C CNN
 F 1 "Micro_SD_Card" H 3200 4450 50  0000 C CNN
-F 2 "10067847-001" H 2800 5350 50  0001 C CNN
+F 2 "mpwifi:MicroSD-slot" H 2800 5350 50  0001 C CNN
 F 3 "" H 2600 5000 50  0000 C CNN
 	1    2600 5000
@@
 F 0 "Q1" H 6650 2025 50  0000 L CNN
 F 1 "BSS138" H 6650 1950 50  0000 L CNN
-F 2 "SOT-23" H 6650 1875 50  0000 L CIN
+F 2 "TO_SOT_Packages_SMD:SOT-23" H 6650 1875 50  0000 L CIN
 F 3 "" H 6450 1950 50  0000 L CNN
 	1    6450 1950
@@
 F 0 "Q2" H 8050 2025 50  0000 L CNN
 F 1 "BSS138" H 8050 1950 50  0000 L CNN
-F 2 "SOT-23" H 8050 1875 50  0000 L CIN
+F 2 "TO_SOT_Packages_SMD:SOT-23" H 8050 1875 50  0000 L CIN
 F 3 "" H 7850 1950 50  0000 L CNN
 	1    7850 1950
@@
 F 0 "R2" V 6630 1250 50  0000 C CNN
 F 1 "10k" V 6550 1250 50  0000 C CNN
-F 2 "" V 6480 1250 50  0000 C CNN
+F 2 "Resistors_SMD:R_0603" V 6480 1250 50  0001 C CNN
 F 3 "" H 6550 1250 50  0000 C CNN
 	1    6550 1250
@@
 F 0 "R3" V 8030 1250 50  0000 C CNN
 F 1 "10k" V 7950 1250 50  0000 C CNN
-F 2 "" V 7880 1250 50  0000 C CNN
+F 2 "Resistors_SMD:R_0603" V 7880 1250 50  0001 C CNN
 F 3 "" H 7950 1250 50  0000 C CNN
 	1    7950 1250
@@
 F 0 "R4" V 6330 2350 50  0000 C CNN
 F 1 "10k" V 6250 2350 50  0000 C CNN
-F 2 "" V 6180 2350 50  0000 C CNN
+F 2 "Resistors_SMD:R_0603" V 6180 2350 50  0001 C CNN
 F 3 "" H 6250 2350 50  0000 C CNN
 	1    6250 2350
@@
 F 0 "R5" V 7730 2350 50  0000 C CNN
 F 1 "10k" V 7650 2350 50  0000 C CNN
-F 2 "" V 7580 2350 50  0000 C CNN
+F 2 "Resistors_SMD:R_0603" V 7580 2350 50  0001 C CNN
 F 3 "" H 7650 2350 50  0000 C CNN
 	1    7650 2350
@@
 L +3.3V #PWR06
 U 1 1 582B7D2E
-P 7050 3800
-F 0 "#PWR06" H 7050 3650 50  0001 C CNN
-F 1 "+3.3V" H 7050 3940 50  0000 C CNN
-F 2 "" H 7050 3800 50  0000 C CNN
-F 3 "" H 7050 3800 50  0000 C CNN
-	1    7050 3800
+P 6600 3650
+F 0 "#PWR06" H 6600 3500 50  0001 C CNN
+F 1 "+3.3V" H 6600 3790 50  0000 C CNN
+F 2 "" H 6600 3650 50  0000 C CNN
+F 3 "" H 6600 3650 50  0000 C CNN
+	1    6600 3650
 	1    0    0    -1
 $EndComp
@@
 F 0 "U1" H 2650 2450 50  0000 C CNN
 F 1 "MCP1703T-3302E/CB" H 2550 2750 50  0000 C CNN
-F 2 "SOT-223-3" H 2800 2350 50  0000 C CNN
-F 3 "" H 2550 2600 50  0000 C CNN
+F 2 "mpwifi:SOT-223-3" H 2800 2350 50  0000 C CNN
+F 3 "http://ww1.microchip.com/downloads/en/DeviceDoc/22049f.pdf" H 2550 2600 50  0001 C CNN
 	1    2550 2600
 	1    0    0    -1
@@
 F 0 "C1" H 1975 3050 50  0000 L CNN
 F 1 "1uF" H 1975 2850 50  0000 L CNN
-F 2 "" H 1988 2800 50  0000 C CNN
+F 2 "Capacitors_SMD:C_0603" H 1988 2800 50  0001 C CNN
 F 3 "" H 1950 2950 50  0000 C CNN
 	1    1950 2950
@@
 F 0 "C2" H 3375 3050 50  0000 L CNN
 F 1 "1uF" H 3375 2850 50  0000 L CNN
-F 2 "" H 3388 2800 50  0000 C CNN
+F 2 "Capacitors_SMD:C_0603" H 3388 2800 50  0001 C CNN
 F 3 "" H 3350 2950 50  0000 C CNN
 	1    3350 2950
@@
 L CONN_01X04 P1
 U 1 1 582BB682
-P 2100 1500
-F 0 "P1" H 2100 1750 50  0000 C CNN
-F 1 "CONN_01X04" V 2200 1500 50  0001 C CNN
-F 2 "" H 2100 1500 50  0000 C CNN
-F 3 "" H 2100 1500 50  0000 C CNN
-	1    2100 1500
-	-1   0    0    -1
+P 2000 1500
+F 0 "P1" H 2000 1750 50  0000 C CNN
+F 1 "CONN_01X04" V 2100 1500 50  0001 C CNN
+F 2 "Socket_Strips:Socket_Strip_Angled_1x04" H 2000 1500 50  0001 C CNN
+F 3 "" H 2000 1500 50  0000 C CNN
+	1    2000 1500
+	-1   0    0    1
 $EndComp
 $Comp
@@
 F 0 "D1" H 1400 2950 50  0000 C CNN
 F 1 "LED" H 1400 2750 50  0000 C CNN
-F 2 "" H 1400 2850 50  0000 C CNN
+F 2 "Diodes_SMD:D_0603" H 1400 2850 50  0001 C CNN
 F 3 "" H 1400 2850 50  0000 C CNN
 	1    1400 2850
@@
 P 1400 3350
 F 0 "R1" V 1480 3350 50  0000 C CNN
-F 1 "R" V 1400 3350 50  0000 C CNN
-F 2 "" V 1330 3350 50  0000 C CNN
+F 1 "140" V 1400 3350 50  0000 C CNN
+F 2 "Resistors_SMD:R_0603" V 1330 3350 50  0001 C CNN
 F 3 "" H 1400 3350 50  0000 C CNN
 	1    1400 3350
@@
 Connection ~ 9300 4300
 Wire Wire Line
-	7050 3800 7600 3800
-Wire Wire Line
-	7050 3800 7050 4300
-Wire Wire Line
-	7050 4300 7600 4300
+	6600 3800 7600 3800
+Wire Wire Line
+	6600 4300 7600 4300
 Wire Wire Line
 	1400 2600 2250 2600
@@
 Connection ~ 3350 2600
 Wire Wire Line
-	2700 1350 2300 1350
-Wire Wire Line
-	2300 1450 3100 1450
+	2200 1350 2700 1350
+Wire Wire Line
+	2200 1450 3100 1450
 Wire Wire Line
 	2550 3200 2550 2800
@@
 	5400 3050 5400 800
 Wire Notes Line
-	6650 3200 9950 3200
+	6300 3200 9950 3200
 Wire Notes Line
 	9950 3200 9950 5400
 Wire Notes Line
-	9950 5400 6650 5400
-Wire Notes Line
-	6650 5400 6650 3200
+	9950 5400 6300 5400
 $Comp
 L CONN_01X03 P2
@@
 F 0 "P2" H 9700 4200 50  0000 C CNN
 F 1 "Flash" V 9800 4000 50  0000 C CNN
-F 2 "" H 9700 4000 50  0000 C CNN
+F 2 "Pin_Headers:Pin_Header_Angled_1x03" H 9700 4000 50  0001 C CNN
 F 3 "" H 9700 4000 50  0000 C CNN
 	1    9700 4000
@@
 	1950 2500 1950 2800
 Wire Wire Line
-	2300 1550 2700 1550
-Wire Wire Line
-	2300 1650 2700 1650
+	2200 1550 2700 1550
+Wire Wire Line
+	2200 1650 2700 1650
 Text Label 2350 1550 0    60   ~ 0
 RX
@@
 RX
 Wire Wire Line
-	2700 1200 2700 1350
+	2700 1350 2700 1200
 Wire Notes Line
 	1150 800  3850 800
@@
 NoConn ~ 7600 4000
 NoConn ~ 7600 4100
-NoConn ~ 7600 4200
 NoConn ~ 8900 4100
 NoConn ~ 8900 3900
@@
 Text Label 3600 4800 0    60   ~ 0
 CS
+Wire Wire Line
+	1700 5300 1600 5300
+Wire Wire Line
+	1600 5300 1600 5800
+Wire Wire Line
+	1600 5800 2300 5800
+Text Label 1650 5800 0    60   ~ 0
+DETECT_SWITCH
+Wire Wire Line
+	6700 4200 7600 4200
+Text Label 6750 4200 0    60   ~ 0
+DETECT_SWITCH
+Wire Wire Line
+	6600 3650 6600 4300
+Connection ~ 6600 3800
+Wire Notes Line
+	6300 5400 6300 3200
+$Comp
+L R R6
+U 1 1 582CF4F1
+P 3500 5650
+F 0 "R6" V 3580 5650 50  0000 C CNN
+F 1 "10k" V 3500 5650 50  0000 C CNN
+F 2 "Resistors_SMD:R_0603" V 3430 5650 50  0001 C CNN
+F 3 "" H 3500 5650 50  0000 C CNN
+	1    3500 5650
+	0    1    1    0
+$EndComp
+Wire Wire Line
+	3350 5650 1600 5650
+Connection ~ 1600 5650
+$Comp
+L +3.3V #PWR024
+U 1 1 582CF62A
+P 3750 5550
+F 0 "#PWR024" H 3750 5400 50  0001 C CNN
+F 1 "+3.3V" H 3750 5690 50  0000 C CNN
+F 2 "" H 3750 5550 50  0000 C CNN
+F 3 "" H 3750 5550 50  0000 C CNN
+	1    3750 5550
+	1    0    0    -1
+$EndComp
+Wire Wire Line
+	3750 5550 3750 5650
+Wire Wire Line
+	3750 5650 3650 5650
 $EndSCHEMATC

Commit message: microSD footprint & retrack
Parts:
- CON1: symbol Micro_SD_Card -> Micro_SD_Card-RESCUE-MPWifi_v1
- D1: symbol LED -> LED-RESCUE-MPWifi_v1
Connections:
- wire segments 78 -> 74
